File: kicad/ledian-support-board/connectors.kicad_sch (KiCad schematic)
At the start: 2 parts, among them J1 Conn_02x13_Odd_Even, J2 Conn_02x13_Odd_Even

Commit message: kicad: ledian-support-board: added titles to all pages
Other:
- title: (none) -> External connectors
Changed lines of the file:
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@@
 (kicad_sch (version 20230121) (generator eeschema)
   (paper "A4")
+  (title_block
+    (title "External connectors")
+  )
   (junction (at 200.66 40.64) (diameter 0) (color 0 0 0 0)
   )
