File: kicad/ledian-support-board/i2c.kicad_sch (KiCad schematic)
At the start: 3 parts, among them U8 BME280

Commit message: kicad: ledian-support-board: added titles to all pages
Other:
- title: (none) -> I2C
Changed lines of the file:
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@@
 (kicad_sch (version 20230121) (generator eeschema)
   (paper "A4")
+  (title_block
+    (title "I2C")
+  )
   (wire (pts (xy 161.29 104.14) (xy 181.61 104.14))
     (stroke (width 0) (type default))
