File: kicad/ledian-support-board/spi.kicad_sch (KiCad schematic)
At the start: 10 parts, among them IC1 SN74HCT125N

Commit message: kicad: ledian-support-board: added titles to all pages
Other:
- title: (none) -> SPI
Changed lines of the file:
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@@
 (kicad_sch (version 20230121) (generator eeschema)
   (paper "A4")
+  (title_block
+    (title "SPI")
+  )
   (junction (at 191.77 97.79) (diameter 0) (color 0 0 0 0)
   )
